File: schematics/v1/jkw_hdmi.sch (EAGLE design)
At the start: 30 parts, among them J1 2X20-CHIP-HEADERS, J2 T_MOLEX_45171, U1 DS2431P

Commit message: layout 1
Connections:
- net VCC_5V_DCC: now also J1.VCC-5V@2; no longer J1.VCC-5V@1
Changed lines of the file:
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@@
-</segment>
-<segment>
-<pinref part="J1" gate="G$1" pin="GND@7"/>
-<wire x1="220.98" y1="71.12" x2="215.9" y2="71.12" width="0.1524" layer="91"/>
 </segment>
 <segment>
@@
 <pinref part="C17" gate="G$1" pin="2"/>
 </segment>
+<segment>
+<pinref part="J1" gate="G$1" pin="GND@7"/>
+<wire x1="220.98" y1="71.12" x2="215.9" y2="71.12" width="0.1524" layer="91"/>
+</segment>
 </net>
 <net name="LCD-D3" class="0">
@@
 <net name="VCC_5V_DCC" class="0">
 <segment>
-<wire x1="137.16" y1="7.62" x2="137.16" y2="93.98" width="0.1524" layer="91"/>
-<pinref part="J1" gate="G$1" pin="VCC-5V@1"/>
-<wire x1="137.16" y1="93.98" x2="157.48" y2="93.98" width="0.1524" layer="91"/>
-<wire x1="137.16" y1="7.62" x2="-116.84" y2="7.62" width="0.1524" layer="91"/>
+<wire x1="271.78" y1="7.62" x2="-116.84" y2="7.62" width="0.1524" layer="91"/>
 <wire x1="-116.84" y1="7.62" x2="-116.84" y2="12.7" width="0.1524" layer="91"/>
 <pinref part="U$2" gate="G$1" pin="VCC5V"/>
@@
 <wire x1="-127" y1="12.7" x2="-116.84" y2="12.7" width="0.1524" layer="91"/>
 <junction x="-116.84" y="12.7"/>
-</segment>
-</net>
+<pinref part="J1" gate="G$1" pin="VCC-5V@2"/>
+<wire x1="254" y1="96.52" x2="271.78" y2="96.52" width="0.1524" layer="91"/>
+<wire x1="271.78" y1="7.62" x2="271.78" y2="96.52" width="0.1524" layer="91"/>
+</segment>
+</net>

Commit message: improved silk
Parts:
- added POWER_USB: USBUSB-MICROB-SMT-DIP, Spark:USBUSB-MICROB-SMT-DIP
- added U$3: LOGO_10X10_SILK, logo:LOGO_10X10_SILK
- added U$4: LOGO_25X25_SILK, logo:LOGO_25X25_SILK
Connections:
- removed net N$1: J1.ACIN-5V
- new net VOUT: J1.ACIN-5V, POWER_USB.VBUS
- net GND: now also POWER_USB.GND
Changed lines of the file:
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@@
 <part name="GND22" library="supply1" deviceset="GND" device=""/>
 <part name="C17" library="rcl" deviceset="C-EU" device="C0805" value="10pF"/>
+<part name="U$3" library="logo" deviceset="LOGO_10X10_SILK" device=""/>
+<part name="U$4" library="logo" deviceset="LOGO_25X25_SILK" device=""/>
+<part name="POWER_USB" library="Spark" deviceset="USB" device="USB-MICROB-SMT-DIP"/>
+<part name="GND23" library="supply1" deviceset="GND" device=""/>
 </parts>
 <sheets>
@@
 <instance part="GND22" gate="1" x="-45.72" y="170.18"/>
 <instance part="C17" gate="G$1" x="-45.72" y="177.8"/>
+<instance part="U$3" gate="G$1" x="-185.42" y="129.54"/>
+<instance part="U$4" gate="G$1" x="-185.42" y="121.92"/>
+<instance part="POWER_USB" gate="G$1" x="223.52" y="134.62"/>
+<instance part="GND23" gate="1" x="215.9" y="129.54"/>
 </instances>
 <busses>
@@
 <wire x1="220.98" y1="71.12" x2="215.9" y2="71.12" width="0.1524" layer="91"/>
 </segment>
+<segment>
+<pinref part="POWER_USB" gate="G$1" pin="GND"/>
+<pinref part="GND23" gate="1" pin="GND"/>
+<wire x1="220.98" y1="134.62" x2="215.9" y2="134.62" width="0.1524" layer="91"/>
+<wire x1="215.9" y1="134.62" x2="215.9" y2="132.08" width="0.1524" layer="91"/>
+</segment>
 </net>
 <net name="LCD-D3" class="0">
@@
 <label x="7.62" y="63.5" size="1.778" layer="95"/>
 <pinref part="U$1" gate="G$1" pin="DE"/>
-</segment>
-</net>
-<net name="N$1" class="0">
-<segment>
-<pinref part="J1" gate="G$1" pin="ACIN-5V"/>
-<wire x1="190.5" y1="96.52" x2="208.28" y2="96.52" width="0.1524" layer="91"/>
 </segment>
 </net>
@@
 </segment>
 </net>
+<net name="VOUT" class="0">
+<segment>
+<pinref part="POWER_USB" gate="G$1" pin="VBUS"/>
+<wire x1="220.98" y1="137.16" x2="203.2" y2="137.16" width="0.1524" layer="91"/>
+<label x="205.74" y="137.16" size="1.778" layer="95"/>
+<pinref part="J1" gate="G$1" pin="ACIN-5V"/>
+<wire x1="190.5" y1="96.52" x2="203.2" y2="96.52" width="0.1524" layer="91"/>
+<wire x1="203.2" y1="137.16" x2="203.2" y2="96.52" width="0.1524" layer="91"/>
+</segment>
+</net>
