File: schematics/v2/jkw_hdmi_v2.brd (EAGLE design)
At the start: 40.9 x 50 mm, 32 parts, among them J1 2X20-CHIP-HEADERS, J2 T_MOLEX_45171, U1 DS2431P

Commit message: added v2 with DCDC
Parts:
- added D6: ES2D, diode:SMB
- added GND, VIN: WIREPAD3,17/1,3, wirepad:3,17/1,3
- added JP1: (no value), jumper:SJ_2
- added U$9: MP1584EN, power_supply:MP1584EN
- moved POWER_USB 13.2 mm to (28.8, 52.8)
- moved R19 2.27 mm to (20.0, 40.6)
- moved C6 1.50 mm to (23.3, 46.1)
- moved C7 1.50 mm to (18.1, 46.1)
- moved L5 1.50 mm to (20.7, 46.1)
- moved C17 1.41 mm to (38.9, 35.6), turned to 0 degrees
- moved C14 1.30 mm to (31.9, 46.2)
- moved C15 1.30 mm to (27.6, 46.2)
- moved L2 1.30 mm to (29.8, 46.2)
- moved C11 0.86 mm to (41.1, 43.5)
- moved L1 0.81 mm to (41.1, 41.4)
- moved C10 0.80 mm to (41.1, 39.3)
- moved R3 0.66 mm to (18.8, 40.2)
- moved R4 0.52 mm to (18.8, 42.2)
Connections:
- new net N$12: J1.CHG-IN, JP1.2
- new net N$65: D6.A, VIN.1
- new net USBV: JP1.1, POWER_USB.VBUS
- new net VIN: D6.C, U$9.VIN
- net GND: now also GND.1, U$9.GNDIN, U$9.GNDOUT
- net VOUT: now also JP1.3, U$9.VOUT; no longer J1.CHG-IN, POWER_USB.VBUS
Routing:
- net GND: track 551.3 -> 580.4 mm, vias 42 -> 45
- net VOUT: track 31.8 -> 4.39 mm
- net TX1-: track 20.9 -> 34.4 mm
- net TX1+: track 22.5 -> 34.4 mm
- net TX2-: track 23.5 -> 34.4 mm
- net TX2+: track 23.6 -> 34.3 mm
- net USBV: track 0.00 -> 10.0 mm
- net TX0-: track 25.2 -> 34.3 mm
- net VIN: track 0.00 -> 9.06 mm, vias 0 -> 1
- net N$65: track 0.00 -> 8.93 mm, vias 0 -> 1
- net TX0+: track 25.5 -> 34.4 mm
- net N$12: track 0.00 -> 7.85 mm
- net VCC: track 189.7 -> 184.2 mm
- net N$5: track 12.3 -> 14.6 mm
- net TXC+: track 32.6 -> 34.4 mm
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
Commit message: added v2 with DCDC
Parts:
- added U$4: LOGO_3X3_COPPER, JKW_CHIP:LOGO_3X3_COPPER
- U$9: value MP1584EN -> MP1584EN_FRAMELESS; device power_supply:MP1584EN -> JKW_CHIP:MP1584EN_FRAMELESS
- moved R3 22.5 mm to (41.2, 38.5)
- moved R4 22.5 mm to (41.2, 40.6)
- moved U$3 0.47 mm to (38.4, 19.5)
Routing:
- net TWI1_SCK: track 44.5 -> 48.3 mm
- net VCC: track 184.2 -> 187.4 mm, vias 11 -> 12
- net TWI1_SDA: track 51.6 -> 53.5 mm
- net GND: track 580.4 -> 579.1 mm
Other:
- board text added: "JKW v2"
