File: schematics/v3_audio/jkw_hdmi_v2.brd (EAGLE design)
At the start: 40.9 x 50 mm, 47 parts, among them J1 2X20-CHIP-HEADERS, J3 T_MOLEX_45171, Q2 12mhz, U1 DS2431P, U2 LP5907MFX

Commit message: routing v1 done
Parts:
- removed U$3: LOGO_10X10_SILK, logo:LOGO_10X10_SILK
- removed USB1: USBUSB-MICROB-SMT-DIP, Spark:USB-MICROB-SMT-DIP
- added AUDIO_USB: USBUSB-MICROB-SMT-DIP, Spark:USB-MICROB-SMT-DIP
- added C1, C2: 100nF, rcl:C0805
- added TP1: TPSQTP12SQ, testpad:TP12SQ
- added U$1: LOGO_25X25_SILK, JKW_CHIP:LOGO_25X25_SILK
- moved C18 18.1 mm to (9.50, 10.5), turned to 180 degrees
- moved C19 17.1 mm to (9.50, 8.43), turned to 180 degrees
- moved C20 16.6 mm to (9.50, 4.29), turned to 0 degrees
- moved L3 16.5 mm to (9.50, 6.38), turned to 180 degrees
- moved JP1 13.6 mm to (5.94, 43.4), flipped to the bottom, turned to 270 degrees
- moved C30 12.2 mm to (25.7, 12.4)
- moved J3 12.2 mm to (21.5, -0.89)
- moved R6 12.2 mm to (21.0, 12.5)
- moved C22 12.2 mm to (10.9, 20.0)
- moved C27 12.2 mm to (7.29, 39.1)
- moved C43 12.2 mm to (28.0, 39.5)
- moved D6 12.2 mm to (32.0, 35.4)
- moved GND 12.2 mm to (32.6, 47.5)
- moved R19 12.2 mm to (9.00, 35.5)
- moved R24 12.2 mm to (21.8, 41.4)
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Connections:
- net 1.8V: now also C1.1, C2.1
- net GND: now also AUDIO_USB.GND, AUDIO_USB.MT1, AUDIO_USB.MT2, C1.2, C2.2; no longer USB1.GND, USB1.MT1, USB1.MT2
- net N$32: now also TP1.TP
- net N$62: now also AUDIO_USB.D+; no longer USB1.D+
- net N$64: now also AUDIO_USB.D-; no longer USB1.D-
- net N$66: now also AUDIO_USB.VBUS; no longer USB1.VBUS
Routing:
- net 1.8V: track 15.2 -> 96.5 mm, vias 5 -> 6
- net GND: track 99.8 -> 139.4 mm, vias 28 -> 51
- net VCC: track 26.6 -> 48.3 mm, vias 5 -> 12
- net N$22: track 0.00 -> 17.2 mm, vias 0 -> 2
- net N$25: track 9.13 -> 23.0 mm, vias 1 -> 0
- net LCD-DE: track 32.4 -> 45.5 mm, vias 1 -> 3
- net N$12: track 0.00 -> 10.4 mm
- net VCC2: track 17.9 -> 26.9 mm, vias 2 -> 3
- net USBV: track 0.00 -> 8.43 mm, vias 0 -> 1
- net VOUT: track 0.00 -> 7.21 mm
- net N$27: track 10.3 -> 17.2 mm, vias 1 -> 0
- net N$5: track 12.1 -> 18.5 mm
- net N$24: track 9.81 -> 15.9 mm, vias 0 -> 2
- net N$1: track 0.00 -> 1.28 mm
- net N$32: track 12.6 -> 13.7 mm
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- added copper zone on layer 2, net GND
- added copper zone on layer 15, net VCC
- added copper zone on layer 16, net VCC2
Other:
- board text added: "JKW v3"
- board text removed: "JKW v2"
