File: schematics/v3_audio/jkw_hdmi_v2.sch (EAGLE design)
At the start: 47 parts, among them J1 2X20-CHIP-HEADERS, J3 T_MOLEX_45171, Q2 12mhz, U1 DS2431P, U2 LP5907MFX

Commit message: routing v1 done
Parts:
- removed U$3: LOGO_10X10_SILK, logo:LOGO_10X10_SILK
- added C1, C2: 100nF, rcl:C-EUC0805
- added TP1: TPSQTP12SQ, testpad:TPSQTP12SQ
- added U$1: LOGO_25X25_SILK, JKW_CHIP:LOGO_25X25_SILK
- renumbered USB1 to AUDIO_USB
Connections:
- net 1.8V: now also C1.1, C2.1
- net GND: now also C1.2, C2.2
- net N$32: now also TP1.TP
Other:
- note added: "Ivdd 80mA IOvdd 0.8mA IAvcc 29mA IPvcc 9mA =90mA@3.3V"
Changed lines of the file:
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@@
 <?xml version="1.0" encoding="utf-8"?>
 <!DOCTYPE eagle SYSTEM "eagle.dtd">
-<eagle version="6.5.0">
+<eagle version="7.6.0">
 <drawing>
 <settings>
@@
 <part name="P+4" library="supply1" deviceset="VCC" device=""/>
 <part name="P+3" library="supply1" deviceset="VCC" device=""/>
-<part name="U$3" library="logo" deviceset="LOGO_10X10_SILK" device=""/>
 <part name="POWER_USB" library="Spark" deviceset="USB" device="USB-MICROB-SMT-DIP"/>
 <part name="GND23" library="supply1" deviceset="GND" device=""/>
@@
 <part name="GND54" library="supply1" deviceset="GND" device=""/>
 <part name="GND55" library="supply1" deviceset="GND" device=""/>
-<part name="USB1" library="Spark" deviceset="USB" device="USB-MICROB-SMT-DIP"/>
+<part name="AUDIO_USB" library="Spark" deviceset="USB" device="USB-MICROB-SMT-DIP"/>
 <part name="R23" library="rcl" deviceset="R-EU_" device="M0805" value="22"/>
 <part name="R24" library="rcl" deviceset="R-EU_" device="M0805" value="22"/>
@@
 <part name="R26" library="rcl" deviceset="R-EU_" device="M0805" value="1k5"/>
 <part name="GND45" library="supply1" deviceset="GND" device=""/>
+<part name="C1" library="rcl" deviceset="C-EU" device="C0805" value="100nF"/>
+<part name="C2" library="rcl" deviceset="C-EU" device="C0805" value="100nF"/>
+<part name="GND1" library="supply1" deviceset="GND" device=""/>
+<part name="GND2" library="supply1" deviceset="GND" device=""/>
+<part name="U$1" library="JKW_CHIP" deviceset="LOGO_25X25_SILK" device=""/>
+<part name="TP1" library="testpad" deviceset="TPSQ" device="TP12SQ"/>
 </parts>
 <sheets>
@@
 <text x="10.16" y="-203.2" size="1.778" layer="91" rot="R90">TODO!</text>
 <text x="-104.14" y="-198.12" size="1.778" layer="91">TODO!</text>
+<text x="48.26" y="-76.2" size="1.778" layer="91">Ivdd 80mA
+IOvdd 0.8mA
+IAvcc 29mA
+IPvcc 9mA
+=90mA@3.3V</text>
 </plain>
 <instances>
@@
 <instance part="P+4" gate="VCC" x="-58.42" y="88.9"/>
 <instance part="P+3" gate="VCC" x="-66.04" y="149.86"/>
-<instance part="U$3" gate="G$1" x="-147.32" y="-264.16"/>
 <instance part="POWER_USB" gate="G$1" x="25.4" y="121.92"/>
 <instance part="GND23" gate="1" x="17.78" y="116.84"/>
@@
 <instance part="GND54" gate="1" x="203.2" y="-114.3" rot="R180"/>
 <instance part="GND55" gate="1" x="187.96" y="-114.3" rot="R180"/>
-<instance part="USB1" gate="G$1" x="246.38" y="-213.36"/>
+<instance part="AUDIO_USB" gate="G$1" x="246.38" y="-213.36"/>
 <instance part="R23" gate="G$1" x="200.66" y="-205.74" rot="R180"/>
 <instance part="R24" gate="G$1" x="200.66" y="-208.28" rot="R180"/>
@@
 <instance part="R26" gate="G$1" x="170.18" y="-152.4"/>
 <instance part="GND45" gate="1" x="226.06" y="-182.88"/>
+<instance part="C1" gate="G$1" x="17.78" y="-121.92"/>
+<instance part="C2" gate="G$1" x="7.62" y="-121.92"/>
+<instance part="GND1" gate="1" x="7.62" y="-132.08"/>
+<instance part="GND2" gate="1" x="17.78" y="-132.08"/>
+<instance part="U$1" gate="G$1" x="-147.32" y="-281.94"/>
+<instance part="TP1" gate="G$1" x="104.14" y="-170.18"/>
 </instances>
 <busses>
@@
 </segment>
 <segment>
-<pinref part="USB1" gate="G$1" pin="GND"/>
+<pinref part="AUDIO_USB" gate="G$1" pin="GND"/>
 <pinref part="GND56" gate="1" pin="GND"/>
 <wire x1="243.84" y1="-213.36" x2="241.3" y2="-213.36" width="0.1524" layer="91"/>
@@
 <wire x1="226.06" y1="-170.18" x2="226.06" y2="-175.26" width="0.1524" layer="91"/>
 <junction x="226.06" y="-175.26"/>
+</segment>
+<segment>
+<pinref part="C2" gate="G$1" pin="2"/>
+<pinref part="GND1" gate="1" pin="GND"/>
+<wire x1="7.62" y1="-129.54" x2="7.62" y2="-127" width="0.1524" layer="91"/>
+</segment>
+<segment>
+<pinref part="C1" gate="G$1" pin="2"/>
+<pinref part="GND2" gate="1" pin="GND"/>
+<wire x1="17.78" y1="-129.54" x2="17.78" y2="-127" width="0.1524" layer="91"/>
 </segment>
 </net>
@@
 <wire x1="17.78" y1="-96.52" x2="17.78" y2="-93.98" width="0.1524" layer="91"/>
 <junction x="17.78" y="-93.98"/>
+<pinref part="C1" gate="G$1" pin="1"/>
+<wire x1="17.78" y1="-119.38" x2="17.78" y2="-116.84" width="0.1524" layer="91"/>
+<wire x1="17.78" y1="-116.84" x2="27.94" y2="-116.84" width="0.1524" layer="91"/>
+<wire x1="27.94" y1="-116.84" x2="27.94" y2="-109.22" width="0.1524" layer="91"/>
+<pinref part="C2" gate="G$1" pin="1"/>
+<wire x1="17.78" y1="-116.84" x2="7.62" y2="-116.84" width="0.1524" layer="91"/>
+<wire x1="7.62" y1="-116.84" x2="7.62" y2="-119.38" width="0.1524" layer="91"/>
+<junction x="17.78" y="-116.84"/>
+<junction x="27.94" y="-109.22"/>
 </segment>
 </net>
@@
 <segment>
 <pinref part="U$6" gate="G$1" pin="SPDIF"/>
-<wire x1="86.36" y1="-167.64" x2="147.32" y2="-167.64" width="0.1524" layer="91"/>
+<wire x1="86.36" y1="-167.64" x2="104.14" y2="-167.64" width="0.1524" layer="91"/>
 <pinref part="U$5" gate="G$1" pin="DOUT"/>
+<wire x1="104.14" y1="-167.64" x2="147.32" y2="-167.64" width="0.1524" layer="91"/>
 <wire x1="147.32" y1="-167.64" x2="147.32" y2="-157.48" width="0.1524" layer="91"/>
 <wire x1="147.32" y1="-157.48" x2="177.8" y2="-157.48" width="0.1524" layer="91"/>
+<pinref part="TP1" gate="G$1" pin="TP"/>
+<junction x="104.14" y="-167.64"/>
 </segment>
 </net>
@@
 <segment>
 <pinref part="R23" gate="G$1" pin="1"/>
-<pinref part="USB1" gate="G$1" pin="D+"/>
+<pinref part="AUDIO_USB" gate="G$1" pin="D+"/>
 <wire x1="205.74" y1="-205.74" x2="215.9" y2="-205.74" width="0.1524" layer="91"/>
 <pinref part="R25" gate="G$1" pin="1"/>
@@
 <segment>
 <pinref part="R24" gate="G$1" pin="1"/>
-<pinref part="USB1" gate="G$1" pin="D-"/>
+<pinref part="AUDIO_USB" gate="G$1" pin="D-"/>
 <wire x1="205.74" y1="-208.28" x2="243.84" y2="-208.28" width="0.1524" layer="91"/>
 </segment>
@@
 <pinref part="U$5" gate="G$1" pin="VBUS"/>
 <wire x1="177.8" y1="-170.18" x2="167.64" y2="-170.18" width="0.1524" layer="91"/>
-<pinref part="USB1" gate="G$1" pin="VBUS"/>
+<pinref part="AUDIO_USB" gate="G$1" pin="VBUS"/>
 <wire x1="243.84" y1="-210.82" x2="226.06" y2="-210.82" width="0.1524" layer="91"/>
 <wire x1="226.06" y1="-210.82" x2="167.64" y2="-210.82" width="0.1524" layer="91"/>
