File: schematics/v3_audio/jkw_hdmi_v3.brd (EAGLE design)
At the start: 40.9 x 50 mm, 51 parts, among them J1 2X20-CHIP-HEADERS, J3 T_MOLEX_45171, Q2 12mhz, U1 DS2431P, U2 LP5907MFX

Commit message: minor fixes
Parts:
- J1: device VGA-DIP:2X20CHIP_SM -> JKW_CHIP:2X20CHIP_SM
- moved C18 5.81 mm to (14.4, 13.6)
- moved C3 1.16 mm to (18.7, 42.0), turned to 180 degrees
- moved C20 0.91 mm to (9.50, 5.21)
- moved L3 0.89 mm to (9.50, 7.26)
- moved C19 0.89 mm to (9.50, 9.32)
- moved R26 0.33 mm to (21.5, 37.3), turned to 180 degrees
Connections:
- net N$12 renamed ACIN
- net N$5 renamed LCD-D2
Routing:
- net VCC: track 79.3 -> 87.4 mm, vias 18 -> 19
- net N$22: track 17.2 -> 24.2 mm
- net N$35: track 13.4 -> 18.7 mm
- net N$27: track 17.2 -> 19.3 mm
- net 1.8V: track 87.7 -> 88.5 mm
- net GND: track 153.0 -> 153.7 mm, vias 52 -> 50
Other:
- board text added: "HDMI JKW v3/2016"
- board text removed: "JKW v3"

Commit message: ?
Parts:
- U2: value LP5907MFX -> LP5907MFX-1.8
Changed lines of the file:
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@@
 <attribute name="VALUE" x="20.7772" y="6.9088" size="1.27" layer="28" rot="MR180"/>
 </element>
-<element name="U2" library="JKW_CHIP" package="SOT23-5" value="LP5907MFX" x="7.3406" y="35.179" smashed="yes">
+<element name="U2" library="JKW_CHIP" package="SOT23-5" value="LP5907MFX-1.8" x="7.3406" y="35.179" smashed="yes">
 <attribute name="VALUE" x="5.789" y="30.7594" size="2.032" layer="27" font="vector" ratio="13" rot="SR0"/>
 </element>
